Commit message: mod

File: legged_gym/resources/robots/g1/g1_custom.urdf (robot description, URDF)
Before this commit: robot g1, 44 links, 43 joints
Joints:
- joint left_shoulder_roll_joint: limit lower=-1.5882 upper=2.2515 effort=21 velocity=53 -> lower=0.0 upper=2.2515 effort=21 velocity=53
- joint right_shoulder_roll_joint: limit lower=-2.2515 upper=1.5882 effort=21 velocity=53 -> lower=-2.2515 upper=0.0 effort=21 velocity=53
